Commit message: First movements in the X-Y Plane

File: scara/scara_ws/src/scara_gz_description/urdf/scara.urdf.xacro (robot description, xacro)
@@ -6,4 +6,8 @@
     <plugin>gz_ros2_control/GazeboSimSystem</plugin>
   </hardware>
+  <joint name="joint_0">
+    <command_interface name="position" />
+    <state_interface name="position" />
+  </joint>
   <joint name="joint_1">
     <command_interface name="position" />
@@ -18,8 +22,4 @@
     <state_interface name="position" />
   </joint>
-  <joint name="joint_4">
-    <command_interface name="position" />
-    <state_interface name="position" />
-  </joint>
 </ros2_control>
 <gazebo>
@@ -27,4 +27,10 @@
   <parameters>$(find scara_gz_bringup)/config/controllers.yaml</parameters>
   </plugin>
+</gazebo>
+<gazebo reference="joint_0">
+  <ros2_control>
+    <command_interface>position</command_interface>
+    <state_interface>position</state_interface>
+  </ros2_control>
 </gazebo>
 <gazebo reference="joint_1">
@@ -46,9 +52,3 @@
   </ros2_control>
 </gazebo>
-<gazebo reference="joint_4">
-  <ros2_control>
-    <command_interface>position</command_interface>
-    <state_interface>position</state_interface>
-  </ros2_control>
-</gazebo>
 </robot>
