Commit message: Just updating

File: abb/abb_ws/install/abb_gz_description/share/abb_gz_description/urdf/common_properties.xacro (robot description, xacro)
@@ -1,42 +1 @@
-<?xml version="1.0"?>
-<robot xmlns:xacro="http://www.ros.org/wiki/xacro">
-    <material name="blue">
-        <color rgba="0 0 0.5 1" />
-    </material>
-    <material name="grey">
-        <color rgba="0.5 0.5 0.5 1" />
-    </material>
-    <material name="orange">
-        <color rgba="1.0 0.5 0 1" />
-    </material>
-    <material name="yellow">
-        <color rgba="1.0 1.0 0 1" />
-    </material>
-    <xacro:macro name="box_inertia" params="m x y z o_xyz o_rpy">
-        <inertial>
-            <mass value="${m}" />
-            <origin xyz="${o_xyz}" rpy="${o_rpy}" />
-            <inertia ixx="${(m/12) * (y*y + z*z)}" ixy="0" ixz="0"
-                     iyy="${(m/12) * (x*x + z*z)}" iyz="0"
-                     izz="${(m/12) * (x*x + y*y)}" />
-        </inertial>
-    </xacro:macro>
-    <xacro:macro name="cylinder_inertia" params="m r l o_xyz o_rpy">
-        <inertial>
-            <mass value="${m}" />
-            <origin xyz="${o_xyz}" rpy="${o_rpy}" />
-            <inertia ixx="${(m/12) * (3*r*r + l*l)}" ixy="0" ixz="0"
-                     iyy="${(m/12) * (3*r*r + l*l)}" iyz="0"
-                     izz="${(m/2) * (r*r)}" />
-        </inertial>
-    </xacro:macro>
-    <xacro:macro name="sphere_inertia" params="m r o_xyz o_rpy">
-        <inertial>
-            <mass value="${m}" />
-            <origin xyz="${o_xyz}" rpy="${o_rpy}" />
-            <inertia ixx="${(2/5) * m * r * r}" ixy="0" ixz="0"
-                     iyy="${(2/5) * m * r * r}" iyz="0"
-                     izz="${(2/5) * m * r * r}" />
-        </inertial>
-    </xacro:macro>
-</robot>
+/home/eia/repo/rbi_2025_2/abb/abb_ws/src/abb_gz_description/urdf/common_properties.xacro

File: abb/abb_ws/install/abb_gz_description/share/abb_gz_description/urdf/irb140.urdf.xacro (robot description, xacro)
@@ -1,74 +1 @@
-<?xml version="1.0"?>
-<robot name="abb_irb140" xmlns:xacro="http://ros.org/wiki/xacro">
-  <xacro:include filename="irb140_description.xacro" />
-<ros2_control name="MyRobot" type="system">
-  <hardware>
-    <plugin>gz_ros2_control/GazeboSimSystem</plugin>
-  </hardware>
-  <joint name="joint_1">
-    <command_interface name="position" />
-    <state_interface name="position" />
-  </joint>
-  <joint name="joint_2">
-    <command_interface name="position" />
-    <state_interface name="position" />
-  </joint>
-  <joint name="joint_3">
-    <command_interface name="position" />
-    <state_interface name="position" />
-  </joint>
-  <joint name="joint_4">
-    <command_interface name="position" />
-    <state_interface name="position" />
-  </joint>
-  <joint name="joint_5">
-    <command_interface name="position" />
-    <state_interface name="position" />
-  </joint>
-  <joint name="joint_6">
-    <command_interface name="position" />
-    <state_interface name="position" />
-  </joint>
-</ros2_control>
-<gazebo>
-  <plugin name="gz_ros2_control::GazeboSimROS2ControlPlugin" filename="libgz_ros2_control-system.so">
-  <parameters>$(find abb_bringup)/config/controllers.yaml</parameters>
-  </plugin>
-</gazebo>
-<gazebo reference="joint_1">
-  <ros2_control>
-    <command_interface>position</command_interface>
-    <state_interface>position</state_interface>
-  </ros2_control>
-</gazebo>
-<gazebo reference="joint_2">
-  <ros2_control>
-    <command_interface>position</command_interface>
-    <state_interface>position</state_interface>
-  </ros2_control>
-</gazebo>
-<gazebo reference="joint_3">
-  <ros2_control>
-    <command_interface>position</command_interface>
-    <state_interface>position</state_interface>
-  </ros2_control>
-</gazebo>
-<gazebo reference="joint_4">
-  <ros2_control>
-    <command_interface>position</command_interface>
-    <state_interface>position</state_interface>
-  </ros2_control>
-</gazebo>
-<gazebo reference="joint_5">
-  <ros2_control>
-    <command_interface>position</command_interface>
-    <state_interface>position</state_interface>
-  </ros2_control>
-</gazebo>
-<gazebo reference="joint_6">
-  <ros2_control>
-    <command_interface>position</command_interface>
-    <state_interface>position</state_interface>
-  </ros2_control>
-</gazebo>
-</robot>
+/home/eia/repo/rbi_2025_2/abb/abb_ws/src/abb_gz_description/urdf/irb140.urdf.xacro

File: abb/abb_ws/install/abb_gz_description/share/abb_gz_description/urdf/irb140_description.xacro (robot description, xacro)
@@ -1,181 +1 @@
-<?xml version="1.0" ?>
-<robot name="abb_irb140"
-       xmlns:xacro="http://ros.org/wiki/xacro">
-    <xacro:include filename="common_properties.xacro" />
-  <link name="base_link">
-    <visual>
-      <origin rpy="0 0 0" xyz="0 0 0"/>
-      <geometry>
-        <mesh filename="package://abb_description/meshes/irb140/visual/base_link.stl"/>
-      </geometry>
-      <material name="abb_orange">
-        <color rgba="1 0.43 0 1"/>
-      </material>
-    </visual>
-    <collision>
-      <geometry>
-        <mesh filename="package://abb_description/meshes/irb140/collision/base_link.stl"/>
-      </geometry>
-      <material name="yellow">
-        <color rgba="0 1 1 1"/>
-      </material>
-    </collision>
-    <xacro:box_inertia m="1000" x="0.5" y="0.5" z="0.5" o_xyz="0 0 0.2" o_rpy="0 0 0" />
-  </link>
-  <link name="link_1">
-    <visual>
-      <origin rpy="0 0 0" xyz="0 0 0"/>
-      <geometry>
-        <mesh filename="package://abb_description/meshes/irb140/visual/link_1.stl"/>
-      </geometry>
-      <material name="abb_orange"/>
-    </visual>
-    <collision>
-      <origin rpy="0 0 0" xyz="0 0 0"/>
-      <geometry>
-        <mesh filename="package://abb_description/meshes/irb140/collision/link_1.stl"/>
-      </geometry>
-      <material name="yellow"/>
-    </collision>
-    <xacro:cylinder_inertia m="1" r="0.15" l="0.5" o_xyz="0 0 0.25" o_rpy="0 0 0" />
-  </link>
-  <link name="link_2">
-    <visual>
-      <origin rpy="0 0 0" xyz="-0.28 0 -1.38"/>
-      <geometry>
-        <mesh filename="package://abb_description/meshes/irb140/visual/link_2.stl"/>
-      </geometry>
-      <material name="abb_orange"/>
-    </visual>
-    <collision>
-      <origin rpy="0 0 0" xyz="-0.28 0 -1.38"/>
-      <geometry>
-        <mesh filename="package://abb_description/meshes/irb140/collision/link_2.stl"/>
-      </geometry>
-      <material name="yellow"/>
-    </collision>
-    <xacro:box_inertia m="1" x="1.42" y="0.2" z="0.2" o_xyz="0.71 0 0" o_rpy="0 0 0" />
-  </link>
-  <link name="link_3">
-    <visual>
-      <origin rpy="0 0 0" xyz="-0.28 0 -2.8"/>
-      <geometry>
-        <mesh filename="package://abb_description/meshes/irb140/visual/link_3.stl"/>
-      </geometry>
-      <material name="abb_orange"/>
-    </visual>
-    <collision>
-      <origin rpy="0 0 0" xyz="-0.28 0 -2.8"/>
-      <geometry>
-        <mesh filename="package://abb_description/meshes/irb140/collision/link_3.stl"/>
-      </geometry>
-      <material name="yellow"/>
-    </collision>
-    <xacro:box_inertia m="1" x="1.49" y="0.15" z="0.15" o_xyz="0.745 0 0" o_rpy="0 0 0" />
-  </link>
-  <link name="link_4">
-    <visual>
-      <origin rpy="0 0 0" xyz="-0.28 0 -2.8"/>
-      <geometry>
-        <mesh filename="package://abb_description/meshes/irb140/visual/link_4.stl"/>
-      </geometry>
-      <material name="abb_orange"/>
-    </visual>
-    <collision>
-      <origin rpy="0 0 0" xyz="-0.28 0 -2.8"/>
-      <geometry>
-        <mesh filename="package://abb_description/meshes/irb140/collision/link_4.stl"/>
-      </geometry>
-      <material name="yellow"/>
-    </collision>
-    <xacro:box_inertia m="1" x="0.1" y="0.1" z="0.1" o_xyz="0 0 0" o_rpy="0 0 0" />
-  </link>
-  <link name="link_5">
-    <visual>
-      <origin rpy="0 0 0" xyz="-1.77 0 -2.8"/>
-      <geometry>
-        <mesh filename="package://abb_description/meshes/irb140/visual/link_5.stl"/>
-      </geometry>
-      <material name="abb_orange"/>
-    </visual>
-    <collision>
-      <origin rpy="0 0 0" xyz="-1.77 0 -2.8"/>
-      <geometry>
-        <mesh filename="package://abb_description/meshes/irb140/collision/link_5.stl"/>
-      </geometry>
-      <material name="yellow"/>
-    </collision>
-    <xacro:cylinder_inertia m="1" r="0.05" l="0.1" o_xyz="0 0 0" o_rpy="0 0 0" />
-  </link>
-  <link name="link_6">
-    <visual>
-      <origin rpy="0 0 0" xyz="-1.77 0 -2.8"/>
-      <geometry>
-        <mesh filename="package://abb_description/meshes/irb140/visual/link_6.stl"/>
-      </geometry>
-      <material name="abb_orange"/>
-    </visual>
-    <collision>
-      <origin rpy="0 0 0" xyz="-1.77 0 -2.8"/>
-      <geometry>
-        <mesh filename="package://abb_description/meshes/irb140/collision/link_6.stl"/>
-      </geometry>
-      <material name="yellow"/>
-    </collision>
-    <xacro:cylinder_inertia m="1" r="0.03" l="0.05" o_xyz="0 0 0" o_rpy="0 0 0" />
-  </link>
-  <link name="tool0"/>
-  <joint name="joint_1" type="revolute">
-    <origin rpy="0 0 0" xyz="0 0 0"/>
-    <parent link="base_link"/>
-    <child link="link_1"/>
-    <axis xyz="0 0 1"/>
-    <limit effort="100" lower="-3.1416" upper="3.1416" velocity="2.618"/>
-  </joint>
-  <joint name="joint_2" type="revolute">
-    <origin rpy="0 0 0" xyz="0.28 0 1.38"/>
-    <parent link="link_1"/>
-    <child link="link_2"/>
-    <axis xyz="0 1 0"/>
-    <limit effort="100" lower="-1.7453" upper="1.9199" velocity="2.618"/>
-  </joint>
-  <joint name="joint_3" type="revolute">
-    <origin rpy="0 0 0" xyz="0 0 1.42"/>
-    <parent link="link_2"/>
-    <child link="link_3"/>
-    <axis xyz="0 1 0"/>
-    <limit effort="100" lower="-1.0472" upper="1.1345" velocity="2.618"/>
-  </joint>
-  <joint name="joint_4" type="revolute">
-    <origin rpy="0 0 0" xyz="0 0 0"/>
-    <parent link="link_3"/>
-    <child link="link_4"/>
-    <axis xyz="1 0 0"/>
-    <limit effort="100" lower="-3.49" upper="3.49" velocity="6.2832"/>
-  </joint>
-  <joint name="joint_5" type="revolute">
-    <origin rpy="0 0 0" xyz="1.49 0 0"/>
-    <parent link="link_4"/>
-    <child link="link_5"/>
-    <axis xyz="0 1 0"/>
-    <limit effort="100" lower="-2.0944" upper="2.0944" velocity="6.2832"/>
-  </joint>
-  <joint name="joint_6" type="revolute">
-    <origin rpy="0 0 0" xyz="0 0 0.02"/>
-    <parent link="link_5"/>
-    <child link="link_6"/>
-    <axis xyz="1 0 0"/>
-    <limit effort="100" lower="-6.9813" upper="6.9813" velocity="7.854"/>
-  </joint>
-  <joint name="joint_6-tool0" type="fixed">
-    <parent link="link_6"/>
-    <child link="tool0"/>
-    <origin rpy="0 1.57079632679 0" xyz="0 0 0"/>
-  </joint>
-  <link name="base"/>
-  <joint name="base_link-base" type="fixed">
-    <origin rpy="0 0 0" xyz="0 0 0"/>
-    <parent link="base_link"/>
-    <child link="base"/>
-  </joint>
-</robot>
+/home/eia/repo/rbi_2025_2/abb/abb_ws/src/abb_gz_description/urdf/irb140_description.xacro

File: abb/abb_ws/install/abb_mujoco_description/share/abb_mujoco_description/urdf/abb_description.urdf.xacro (robot description, xacro)
@@ -1,98 +1 @@
-<?xml version="1.0"?>
-<robot name="rover" xmlns:xacro="http://www.ros.org/wiki/xacro">
-  <!-- Main body -->
-  <link name="hull_link">
-    <visual>
-      <geometry>
-        <box size="0.6 0.4 0.2"/>
-      </geometry>
-      <material name="blue">
-        <color rgba="0.1 0.1 0.8 1"/>
-      </material>
-    </visual>
-    <collision>
-      <geometry>
-        <box size="0.6 0.4 0.2"/>
-      </geometry>
-    </collision>
-    <inertial>
-      <mass value="10"/>
-      <origin xyz="0 0 0"/>
-      <inertia ixx="1" ixy="0" ixz="0" iyy="1" iyz="0" izz="1"/>
-    </inertial>
-  </link>
-  <!-- Six thruster joints (effort controlled) -->
-  <!-- X, Y, Z, Roll, Pitch, Yaw -->
-  <joint name="thruster_joint_1" type="continuous">
-    <parent link="hull_link"/>
-    <child link="thruster_link_1"/>
-    <origin xyz="0.3 0 0" rpy="0 0 0"/>
-    <axis xyz="1 0 0"/>
-  </joint>
-  <link name="thruster_link_1"/>
-  <joint name="thruster_joint_2" type="continuous">
-    <parent link="hull_link"/>
-    <child link="thruster_link_2"/>
-    <origin xyz="-0.3 0 0" rpy="0 0 0"/>
-    <axis xyz="0 1 0"/>
-  </joint>
-  <link name="thruster_link_2"/>
-  <joint name="thruster_joint_3" type="continuous">
-    <parent link="hull_link"/>
-    <child link="thruster_link_3"/>
-    <origin xyz="0 0 0.1" rpy="0 0 0"/>
-    <axis xyz="0 0 1"/>
-  </joint>
-  <link name="thruster_link_3"/>
-  <joint name="thruster_joint_4" type="continuous">
-    <parent link="hull_link"/>
-    <child link="thruster_link_4"/>
-    <origin xyz="0 0.2 0" rpy="0 0 0"/>
-    <axis xyz="1 0 0"/>
-  </joint>
-  <link name="thruster_link_4"/>
-  <joint name="thruster_joint_5" type="continuous">
-    <parent link="hull_link"/>
-    <child link="thruster_link_5"/>
-    <origin xyz="0 -0.2 0" rpy="0 0 0"/>
-    <axis xyz="0 1 0"/>
-  </joint>
-  <link name="thruster_link_5"/>
-  <joint name="thruster_joint_6" type="continuous">
-    <parent link="hull_link"/>
-    <child link="thruster_link_6"/>
-    <origin xyz="0 0 0.2" rpy="0 0 0"/>
-    <axis xyz="0 0 1"/>
-  </joint>
-  <link name="thruster_link_6"/>
-  <!-- ros2_control tag for hardware interface -->
-  <ros2_control name="abb_control" type="system">
-    <hardware>
-      <plugin>abb_simulator_layer/AbbSimulatorInterface</plugin>
-    </hardware>
-    <joint name="thruster_joint_1">
-      <command_interface name="effort"/>
-      <state_interface name="effort"/>
-    </joint>
-    <joint name="thruster_joint_2">
-      <command_interface name="effort"/>
-      <state_interface name="effort"/>
-    </joint>
-    <joint name="thruster_joint_3">
-      <command_interface name="effort"/>
-      <state_interface name="effort"/>
-    </joint>
-    <joint name="thruster_joint_4">
-      <command_interface name="effort"/>
-      <state_interface name="effort"/>
-    </joint>
-    <joint name="thruster_joint_5">
-      <command_interface name="effort"/>
-      <state_interface name="effort"/>
-    </joint>
-    <joint name="thruster_joint_6">
-      <command_interface name="effort"/>
-      <state_interface name="effort"/>
-    </joint>
-  </ros2_control>
-</robot>
+/home/eia/repo/rbi_2025_2/abb/abb_ws/src/abb_mujoco_description/urdf/abb_description.urdf.xacro

File: abb/abb_ws/install/abb_mujoco_description/share/abb_mujoco_description/urdf/common_properties.xacro (robot description, xacro)
@@ -1,15 +1 @@
-<?xml version="1.0"?>
-<robot xmlns:xacro="http://www.ros.org/wiki/xacro">
-    <material name="blue">
-        <color rgba="0 0 0.5 1" />
-    </material>
-    <material name="grey">
-        <color rgba="0.5 0.5 0.5 1" />
-    </material>
-    <material name="orange">
-        <color rgba="1.0 0.5 0 1" />
-    </material>
-    <material name="yellow">
-        <color rgba="1.0 1.0 0 1" />
-    </material>
-</robot>
+/home/eia/repo/rbi_2025_2/abb/abb_ws/src/abb_mujoco_description/urdf/common_properties.xacro

File: abb/abb_ws/src/abb_gz_description/urdf/irb140.urdf.xacro (robot description, xacro)
@@ -33,5 +33,5 @@
 <gazebo>
   <plugin name="gz_ros2_control::GazeboSimROS2ControlPlugin" filename="libgz_ros2_control-system.so">
-  <parameters>$(find abb_bringup)/config/controllers.yaml</parameters>
+  <parameters>$(find abb_gz_bringup)/config/controllers.yaml</parameters>
   </plugin>
 </gazebo>

File: abb/abb_ws/src/abb_gz_description/urdf/irb140_description.xacro (robot description, xacro)
@@ -7,5 +7,5 @@
       <origin rpy="0 0 0" xyz="0 0 0"/>
       <geometry>
-        <mesh filename="package://abb_description/meshes/irb140/visual/base_link.stl"/>
+        <mesh filename="package://abb_gz_description/meshes/irb140/visual/base_link.stl"/>
       </geometry>
       <material name="abb_orange">
@@ -15,5 +15,5 @@
     <collision>
       <geometry>
-        <mesh filename="package://abb_description/meshes/irb140/collision/base_link.stl"/>
+        <mesh filename="package://abb_gz_description/meshes/irb140/collision/base_link.stl"/>
       </geometry>
       <material name="yellow">
@@ -27,5 +27,5 @@
       <origin rpy="0 0 0" xyz="0 0 0"/>
       <geometry>
-        <mesh filename="package://abb_description/meshes/irb140/visual/link_1.stl"/>
+        <mesh filename="package://abb_gz_description/meshes/irb140/visual/link_1.stl"/>
       </geometry>
       <material name="abb_orange"/>
@@ -34,5 +34,5 @@
       <origin rpy="0 0 0" xyz="0 0 0"/>
       <geometry>
-        <mesh filename="package://abb_description/meshes/irb140/collision/link_1.stl"/>
+        <mesh filename="package://abb_gz_description/meshes/irb140/collision/link_1.stl"/>
       </geometry>
       <material name="yellow"/>
@@ -44,5 +44,5 @@
       <origin rpy="0 0 0" xyz="-0.28 0 -1.38"/>
       <geometry>
-        <mesh filename="package://abb_description/meshes/irb140/visual/link_2.stl"/>
+        <mesh filename="package://abb_gz_description/meshes/irb140/visual/link_2.stl"/>
       </geometry>
       <material name="abb_orange"/>
@@ -51,5 +51,5 @@
       <origin rpy="0 0 0" xyz="-0.28 0 -1.38"/>
       <geometry>
-        <mesh filename="package://abb_description/meshes/irb140/collision/link_2.stl"/>
+        <mesh filename="package://abb_gz_description/meshes/irb140/collision/link_2.stl"/>
       </geometry>
       <material name="yellow"/>
@@ -61,5 +61,5 @@
       <origin rpy="0 0 0" xyz="-0.28 0 -2.8"/>
       <geometry>
-        <mesh filename="package://abb_description/meshes/irb140/visual/link_3.stl"/>
+        <mesh filename="package://abb_gz_description/meshes/irb140/visual/link_3.stl"/>
       </geometry>
       <material name="abb_orange"/>
@@ -68,5 +68,5 @@
       <origin rpy="0 0 0" xyz="-0.28 0 -2.8"/>
       <geometry>
-        <mesh filename="package://abb_description/meshes/irb140/collision/link_3.stl"/>
+        <mesh filename="package://abb_gz_description/meshes/irb140/collision/link_3.stl"/>
       </geometry>
       <material name="yellow"/>
@@ -78,5 +78,5 @@
       <origin rpy="0 0 0" xyz="-0.28 0 -2.8"/>
       <geometry>
-        <mesh filename="package://abb_description/meshes/irb140/visual/link_4.stl"/>
+        <mesh filename="package://abb_gz_description/meshes/irb140/visual/link_4.stl"/>
       </geometry>
       <material name="abb_orange"/>
@@ -85,5 +85,5 @@
       <origin rpy="0 0 0" xyz="-0.28 0 -2.8"/>
       <geometry>
-        <mesh filename="package://abb_description/meshes/irb140/collision/link_4.stl"/>
+        <mesh filename="package://abb_gz_description/meshes/irb140/collision/link_4.stl"/>
       </geometry>
       <material name="yellow"/>
@@ -95,5 +95,5 @@
       <origin rpy="0 0 0" xyz="-1.77 0 -2.8"/>
       <geometry>
-        <mesh filename="package://abb_description/meshes/irb140/visual/link_5.stl"/>
+        <mesh filename="package://abb_gz_description/meshes/irb140/visual/link_5.stl"/>
       </geometry>
       <material name="abb_orange"/>
@@ -102,5 +102,5 @@
       <origin rpy="0 0 0" xyz="-1.77 0 -2.8"/>
       <geometry>
-        <mesh filename="package://abb_description/meshes/irb140/collision/link_5.stl"/>
+        <mesh filename="package://abb_gz_description/meshes/irb140/collision/link_5.stl"/>
       </geometry>
       <material name="yellow"/>
@@ -112,5 +112,5 @@
       <origin rpy="0 0 0" xyz="-1.77 0 -2.8"/>
       <geometry>
-        <mesh filename="package://abb_description/meshes/irb140/visual/link_6.stl"/>
+        <mesh filename="package://abb_gz_description/meshes/irb140/visual/link_6.stl"/>
       </geometry>
       <material name="abb_orange"/>
@@ -119,5 +119,5 @@
       <origin rpy="0 0 0" xyz="-1.77 0 -2.8"/>
       <geometry>
-        <mesh filename="package://abb_description/meshes/irb140/collision/link_6.stl"/>
+        <mesh filename="package://abb_gz_description/meshes/irb140/collision/link_6.stl"/>
       </geometry>
       <material name="yellow"/>
@@ -125,5 +125,5 @@
     <xacro:cylinder_inertia m="1" r="0.03" l="0.05" o_xyz="0 0 0" o_rpy="0 0 0" />
   </link>
-  <link name="tool0"/>
+  <link name="end_effector"/>
   <joint name="joint_1" type="revolute">
     <origin rpy="0 0 0" xyz="0 0 0"/>
@@ -168,7 +168,7 @@
     <limit effort="100" lower="-6.9813" upper="6.9813" velocity="7.854"/>
   </joint>
-  <joint name="joint_6-tool0" type="fixed">
+  <joint name="joint_6-end_effector" type="fixed">
     <parent link="link_6"/>
-    <child link="tool0"/>
+    <child link="end_effector"/>
     <origin rpy="0 1.57079632679 0" xyz="0 0 0"/>
   </joint>

File: rov/rov_ws/install/rov_mujoco_description/share/rov_mujoco_description/urdf/common_properties.xacro (robot description, xacro)
@@ -1,15 +1 @@
-<?xml version="1.0"?>
-<robot xmlns:xacro="http://www.ros.org/wiki/xacro">
-    <material name="blue">
-        <color rgba="0 0 0.5 1" />
-    </material>
-    <material name="grey">
-        <color rgba="0.5 0.5 0.5 1" />
-    </material>
-    <material name="orange">
-        <color rgba="1.0 0.5 0 1" />
-    </material>
-    <material name="yellow">
-        <color rgba="1.0 1.0 0 1" />
-    </material>
-</robot>
+/home/eia/repo/rbi_2025_2/rov/rov_ws/src/rov_mujoco_description/urdf/common_properties.xacro
