Commit message: Just updating

File: rov/rov_ws/install/rov_mujoco_description/share/rov_mujoco_description/urdf/rov_description.urdf.xacro (robot description, xacro)
@@ -1,98 +1 @@
-<?xml version="1.0"?>
-<robot name="rover" xmlns:xacro="http://www.ros.org/wiki/xacro">
-  <!-- Main body -->
-  <link name="hull_link">
-    <visual>
-      <geometry>
-        <box size="0.6 0.4 0.2"/>
-      </geometry>
-      <material name="blue">
-        <color rgba="0.1 0.1 0.8 1"/>
-      </material>
-    </visual>
-    <collision>
-      <geometry>
-        <box size="0.6 0.4 0.2"/>
-      </geometry>
-    </collision>
-    <inertial>
-      <mass value="10"/>
-      <origin xyz="0 0 0"/>
-      <inertia ixx="1" ixy="0" ixz="0" iyy="1" iyz="0" izz="1"/>
-    </inertial>
-  </link>
-  <!-- Six thruster joints (effort controlled) -->
-  <!-- X, Y, Z, Roll, Pitch, Yaw -->
-  <joint name="thruster_joint_1" type="continuous">
-    <parent link="hull_link"/>
-    <child link="thruster_link_1"/>
-    <origin xyz="0.3 0 0" rpy="0 0 0"/>
-    <axis xyz="1 0 0"/>
-  </joint>
-  <link name="thruster_link_1"/>
-  <joint name="thruster_joint_2" type="continuous">
-    <parent link="hull_link"/>
-    <child link="thruster_link_2"/>
-    <origin xyz="-0.3 0 0" rpy="0 0 0"/>
-    <axis xyz="0 1 0"/>
-  </joint>
-  <link name="thruster_link_2"/>
-  <joint name="thruster_joint_3" type="continuous">
-    <parent link="hull_link"/>
-    <child link="thruster_link_3"/>
-    <origin xyz="0 0 0.1" rpy="0 0 0"/>
-    <axis xyz="0 0 1"/>
-  </joint>
-  <link name="thruster_link_3"/>
-  <joint name="thruster_joint_4" type="continuous">
-    <parent link="hull_link"/>
-    <child link="thruster_link_4"/>
-    <origin xyz="0 0.2 0" rpy="0 0 0"/>
-    <axis xyz="1 0 0"/>
-  </joint>
-  <link name="thruster_link_4"/>
-  <joint name="thruster_joint_5" type="continuous">
-    <parent link="hull_link"/>
-    <child link="thruster_link_5"/>
-    <origin xyz="0 -0.2 0" rpy="0 0 0"/>
-    <axis xyz="0 1 0"/>
-  </joint>
-  <link name="thruster_link_5"/>
-  <joint name="thruster_joint_6" type="continuous">
-    <parent link="hull_link"/>
-    <child link="thruster_link_6"/>
-    <origin xyz="0 0 0.2" rpy="0 0 0"/>
-    <axis xyz="0 0 1"/>
-  </joint>
-  <link name="thruster_link_6"/>
-  <!-- ros2_control tag for hardware interface -->
-  <ros2_control name="rov_control" type="system">
-    <hardware>
-      <plugin>rov_simulator_layer/RovSimulatorInterface</plugin>
-    </hardware>
-    <joint name="thruster_joint_1">
-      <command_interface name="effort"/>
-      <state_interface name="effort"/>
-    </joint>
-    <joint name="thruster_joint_2">
-      <command_interface name="effort"/>
-      <state_interface name="effort"/>
-    </joint>
-    <joint name="thruster_joint_3">
-      <command_interface name="effort"/>
-      <state_interface name="effort"/>
-    </joint>
-    <joint name="thruster_joint_4">
-      <command_interface name="effort"/>
-      <state_interface name="effort"/>
-    </joint>
-    <joint name="thruster_joint_5">
-      <command_interface name="effort"/>
-      <state_interface name="effort"/>
-    </joint>
-    <joint name="thruster_joint_6">
-      <command_interface name="effort"/>
-      <state_interface name="effort"/>
-    </joint>
-  </ros2_control>
-</robot>
+/home/eia/repo/rbi_2025_2/rov/rov_ws/src/rov_mujoco_description/urdf/rov_description.urdf.xacro

File: scara/scara_ws/install/scara_gz_description/share/scara_gz_description/urdf/common_properties.xacro (robot description, xacro)
@@ -1,42 +1 @@
-<?xml version="1.0"?>
-<robot xmlns:xacro="http://www.ros.org/wiki/xacro">
-    <material name="blue">
-        <color rgba="0 0 0.5 1" />
-    </material>
-    <material name="grey">
-        <color rgba="0.5 0.5 0.5 1" />
-    </material>
-    <material name="orange">
-        <color rgba="1.0 0.5 0 1" />
-    </material>
-    <material name="yellow">
-        <color rgba="1.0 1.0 0 1" />
-    </material>
-    <xacro:macro name="box_inertia" params="m x y z o_xyz o_rpy">
-        <inertial>
-            <mass value="${m}" />
-            <origin xyz="${o_xyz}" rpy="${o_rpy}" />
-            <inertia ixx="${(m/12) * (y*y + z*z)}" ixy="0" ixz="0"
-                     iyy="${(m/12) * (x*x + z*z)}" iyz="0"
-                     izz="${(m/12) * (x*x + y*y)}" />
-        </inertial>
-    </xacro:macro>
-    <xacro:macro name="cylinder_inertia" params="m r l o_xyz o_rpy">
-        <inertial>
-            <mass value="${m}" />
-            <origin xyz="${o_xyz}" rpy="${o_rpy}" />
-            <inertia ixx="${(m/12) * (3*r*r + l*l)}" ixy="0" ixz="0"
-                     iyy="${(m/12) * (3*r*r + l*l)}" iyz="0"
-                     izz="${(m/2) * (r*r)}" />
-        </inertial>
-    </xacro:macro>
-    <xacro:macro name="sphere_inertia" params="m r o_xyz o_rpy">
-        <inertial>
-            <mass value="${m}" />
-            <origin xyz="${o_xyz}" rpy="${o_rpy}" />
-            <inertia ixx="${(2/5) * m * r * r}" ixy="0" ixz="0"
-                     iyy="${(2/5) * m * r * r}" iyz="0"
-                     izz="${(2/5) * m * r * r}" />
-        </inertial>
-    </xacro:macro>
-</robot>
+/home/eia/repo/rbi_2025_2/scara/scara_ws/src/scara_gz_description/urdf/common_properties.xacro

File: scara/scara_ws/install/scara_gz_description/share/scara_gz_description/urdf/scara.urdf.xacro (robot description, xacro)
@@ -1,54 +1 @@
-<?xml version="1.0"?>
-<robot name="scara" xmlns:xacro="http://ros.org/wiki/xacro">
-  <xacro:include filename="scara_description.xacro" />
-<ros2_control name="Scara" type="system">
-  <hardware>
-    <plugin>gz_ros2_control/GazeboSimSystem</plugin>
-  </hardware>
-  <joint name="joint_1">
-    <command_interface name="position" />
-    <state_interface name="position" />
-  </joint>
-  <joint name="joint_2">
-    <command_interface name="position" />
-    <state_interface name="position" />
-  </joint>
-  <joint name="joint_3">
-    <command_interface name="position" />
-    <state_interface name="position" />
-  </joint>
-  <joint name="joint_4">
-    <command_interface name="position" />
-    <state_interface name="position" />
-  </joint>
-</ros2_control>
-<gazebo>
-  <plugin name="gz_ros2_control::GazeboSimROS2ControlPlugin" filename="libgz_ros2_control-system.so">
-  <parameters>$(find scara_gz_bringup)/config/controllers.yaml</parameters>
-  </plugin>
-</gazebo>
-<gazebo reference="joint_1">
-  <ros2_control>
-    <command_interface>position</command_interface>
-    <state_interface>position</state_interface>
-  </ros2_control>
-</gazebo>
-<gazebo reference="joint_2">
-  <ros2_control>
-    <command_interface>position</command_interface>
-    <state_interface>position</state_interface>
-  </ros2_control>
-</gazebo>
-<gazebo reference="joint_3">
-  <ros2_control>
-    <command_interface>position</command_interface>
-    <state_interface>position</state_interface>
-  </ros2_control>
-</gazebo>
-<gazebo reference="joint_4">
-  <ros2_control>
-    <command_interface>position</command_interface>
-    <state_interface>position</state_interface>
-  </ros2_control>
-</gazebo>
-</robot>
+/home/eia/repo/rbi_2025_2/scara/scara_ws/src/scara_gz_description/urdf/scara.urdf.xacro

File: scara/scara_ws/install/scara_gz_description/share/scara_gz_description/urdf/scara_description.xacro (robot description, xacro)
@@ -1,176 +1 @@
-<?xml version="1.0"?>
-<robot name="scara_urdf" xmlns:xacro="http://www.ros.org/wiki/xacro">
-  <!-- Materials (just for visuals) -->
-  <material name="red"><color rgba="1 0 0 1"/></material>
-  <material name="blue"><color rgba="0 0 1 1"/></material>
-  <material name="green"><color rgba="0 1 0 1"/></material>
-  <material name="gray"><color rgba="0.5 0.5 0.5 1"/></material>
-  <!-- ============== Base ============== -->
-  <link name="scara_base_link">
-    <inertial>
-      <origin xyz="0 0 0" rpy="0 0 0"/>
-      <mass value="10000.0"/>
-      <inertia ixx="0.002" ixy="0" ixz="0" iyy="0.002" iyz="0" izz="0.002"/>
-    </inertial>
-    <visual>
-      <origin xyz="0 0 0" rpy="0 0 0"/>
-      <geometry>
-        <box size="0.2 0.2 0.1"/>
-      </geometry>
-      <material name="red"/>
-    </visual>
-    <collision>
-      <origin xyz="0 0 0" rpy="0 0 0"/>
-      <geometry>
-        <box size="0.2 0.2 0.1"/>
-      </geometry>
-    </collision>
-  </link>
-  <joint name="joint_1" type="revolute">
-    <parent link="scara_base_link"/>
-    <child  link="link1"/>
-    <origin xyz="0 0 0.254" rpy="0 0 0"/>
-    <axis xyz="0 0 1"/>
-    <limit lower="-3.1416" upper="3.1416" effort="50" velocity="3.0"/>
-  </joint>
-  <link name="link1">
-    <inertial>
-      <origin xyz="0 0 0" rpy="0 0 0"/>
-      <mass value="0.5"/>
-      <inertia ixx="0.001" ixy="0" ixz="0" iyy="0.001" iyz="0" izz="0.001"/>
-    </inertial>
-    <visual>
-      <origin xyz="0 0 -0.1" rpy="0 0 0"/>
-      <geometry>
-        <cylinder radius="0.1" length="0.20"/>
-      </geometry>
-      <material name="blue"/>
-    </visual>
-    <collision>
-      <origin xyz="0 0 -0.1" rpy="0 0 0"/>
-      <geometry>
-        <cylinder radius="0.1" length="0.20"/>
-      </geometry>
-    </collision>
-    <visual>
-      <origin xyz="0.08 0 0.025" rpy="0 0 0"/>
-      <geometry>
-        <box size="0.36 0.10 0.04"/>
-      </geometry>
-      <material name="red"/>
-    </visual>
-    <collision>
-      <origin xyz="0.08 0 0.025" rpy="0 0 0"/>
-      <geometry>
-        <box size="0.36 0.10 0.04"/>
-      </geometry>
-    </collision>
-  </link>
-  <joint name="joint_2" type="revolute">
-    <parent link="link1"/>
-    <child  link="link2"/>
-    <origin xyz="0.210 0 0" rpy="0 0 0"/>
-    <axis xyz="0 0 1"/>
-    <limit lower="-3.1416" upper="3.1416" effort="50" velocity="3.0"/>
-  </joint>
-  <link name="link2">
-    <inertial>
-      <origin xyz="0 0 0" rpy="0 0 0"/>
-      <mass value="0.4"/>
-      <inertia ixx="0.001" ixy="0" ixz="0" iyy="0.001" iyz="0" izz="0.001"/>
-    </inertial>
-    <visual>
-      <origin xyz="0 0 0.1" rpy="0 0 0"/>
-      <geometry>
-        <cylinder radius="0.05" length="0.10"/>
-      </geometry>
-      <material name="blue"/>
-    </visual>
-    <collision>
-      <origin xyz="0 0 0.1" rpy="0 0 0"/>
-      <geometry>
-        <cylinder radius="0.05" length="0.10"/>
-      </geometry>
-    </collision>
-    <visual>
-      <origin xyz="0.07 0 0.175" rpy="0 0 0"/>
-      <geometry>
-        <box size="0.26 0.10 0.04"/>
-      </geometry>
-      <material name="red"/>
-    </visual>
-    <collision>
-      <origin xyz="0.07 0 0.175" rpy="0 0 0"/>
-      <geometry>
-        <box size="0.26 0.10 0.04"/>
-      </geometry>
-    </collision>
-    <visual>
-      <origin xyz="0.145 0 0.3" rpy="0 0 0"/>
-      <geometry>
-        <box size="0.10 0.10 0.20"/>
-      </geometry>
-      <material name="red"/>
-    </visual>
-    <collision>
-      <origin xyz="0.145 0 0.3" rpy="0 0 0"/>
-      <geometry>
-        <box size="0.10 0.10 0.20"/>
-      </geometry>
-    </collision>
-  </link>
-  <joint name="joint_3" type="revolute">
-    <parent link="link2"/>
-    <child  link="link3"/>
-    <origin xyz="0.250 0 0" rpy="0 0 0"/>
-    <axis xyz="0 0 1"/>
-    <limit lower="-3.1416" upper="3.1416" effort="50" velocity="3.0"/>
-  </joint>
-  <link name="link3">
-    <inertial>
-      <origin xyz="0 0 0" rpy="0 0 0"/>
-      <mass value="0.3"/>
-      <inertia ixx="0.0008" ixy="0" ixz="0" iyy="0.0008" iyz="0" izz="0.0008"/>
-    </inertial>
-    <visual>
-      <origin xyz="0 0 0.3" rpy="0 0 0"/>
-      <geometry>
-        <cylinder radius="0.05" length="0.10"/>
-      </geometry>
-      <material name="blue"/>
-    </visual>
-    <collision>
-      <origin xyz="0 0 0.3" rpy="0 0 0"/>
-      <geometry>
-        <cylinder radius="0.05" length="0.10"/>
-      </geometry>
-    </collision>
-  </link>
-  <joint name="joint_4" type="prismatic">
-    <parent link="link3"/>
-    <child  link="ee_link"/>
-    <origin xyz="0 0 0" rpy="0 0 0"/>
-    <axis xyz="0 0 1"/>
-    <limit lower="-0.3" upper="0.1" effort="200" velocity="0.5"/>
-  </joint>
-  <link name="ee_link">
-    <inertial>
-      <origin xyz="0 0 0" rpy="0 0 0"/>
-      <mass value="0.2"/>
-      <inertia ixx="0.0005" ixy="0" ixz="0" iyy="0.0005" iyz="0" izz="0.0005"/>
-    </inertial>
-    <visual>
-      <origin xyz="0 0 0.1" rpy="0 0 0"/>
-      <geometry>
-        <box size="0.04 0.04 0.20"/>
-      </geometry>
-      <material name="green"/>
-    </visual>
-    <collision>
-      <origin xyz="0 0 0.1" rpy="0 0 0"/>
-      <geometry>
-        <box size="0.04 0.04 0.20"/>
-      </geometry>
-    </collision>
-  </link>
-</robot>
+/home/eia/repo/rbi_2025_2/scara/scara_ws/src/scara_gz_description/urdf/scara_description.xacro

File: scara/scara_ws/install/scara_mujoco_description/share/scara_mujoco_description/urdf/common_properties.xacro (robot description, xacro)
@@ -1,15 +1 @@
-<?xml version="1.0"?>
-<robot xmlns:xacro="http://www.ros.org/wiki/xacro">
-    <material name="blue">
-        <color rgba="0 0 0.5 1" />
-    </material>
-    <material name="grey">
-        <color rgba="0.5 0.5 0.5 1" />
-    </material>
-    <material name="orange">
-        <color rgba="1.0 0.5 0 1" />
-    </material>
-    <material name="yellow">
-        <color rgba="1.0 1.0 0 1" />
-    </material>
-</robot>
+/home/eia/repo/rbi_2025_2/scara/scara_ws/src/scara_mujoco_description/urdf/common_properties.xacro

File: scara/scara_ws/install/scara_mujoco_description/share/scara_mujoco_description/urdf/scara_description.urdf.xacro (robot description, xacro)
@@ -1,90 +1 @@
-<?xml version="1.0"?>
-<robot name="rover" xmlns:xacro="http://www.ros.org/wiki/xacro">
-  <!-- Main body -->
-  <link name="hull_link">
-    <visual>
-      <geometry>
-        <box size="0.6 0.4 0.2"/>
-      </geometry>
-      <material name="blue">
-        <color rgba="0.1 0.1 0.8 1"/>
-      </material>
-    </visual>
-    <collision>
-      <geometry>
-        <box size="0.6 0.4 0.2"/>
-      </geometry>
-    </collision>
-    <inertial>
-      <mass value="10"/>
-      <origin xyz="0 0 0"/>
-      <inertia ixx="1" ixy="0" ixz="0" iyy="1" iyz="0" izz="1"/>
-    </inertial>
-  </link>
-  <!-- Six thruster joints (effort controlled) -->
-  <!-- X, Y, Z, Roll, Pitch, Yaw -->
-  <joint name="thruster_joint_1" type="continuous">
-    <parent link="hull_link"/>
-    <child link="thruster_link_1"/>
-    <origin xyz="0.3 0 0" rpy="0 0 0"/>
-    <axis xyz="1 0 0"/>
-  </joint>
-  <link name="thruster_link_1"/>
-  <joint name="thruster_joint_2" type="continuous">
-    <parent link="hull_link"/>
-    <child link="thruster_link_2"/>
-    <origin xyz="-0.3 0 0" rpy="0 0 0"/>
-    <axis xyz="0 1 0"/>
-  </joint>
-  <link name="thruster_link_2"/>
-  <joint name="thruster_joint_3" type="continuous">
-    <parent link="hull_link"/>
-    <child link="thruster_link_3"/>
-    <origin xyz="0 0 0.1" rpy="0 0 0"/>
-    <axis xyz="0 0 1"/>
-  </joint>
-  <link name="thruster_link_3"/>
-  <joint name="thruster_joint_4" type="continuous">
-    <parent link="hull_link"/>
-    <child link="thruster_link_4"/>
-    <origin xyz="0 0.2 0" rpy="0 0 0"/>
-    <axis xyz="1 0 0"/>
-  </joint>
-  <link name="thruster_link_4"/>
-  <joint name="thruster_joint_5" type="continuous">
-    <parent link="hull_link"/>
-    <child link="thruster_link_5"/>
-    <origin xyz="0 -0.2 0" rpy="0 0 0"/>
-    <axis xyz="0 1 0"/>
-  </joint>
-  <link name="thruster_link_5"/>
-  <joint name="thruster_joint_6" type="continuous">
-    <parent link="hull_link"/>
-    <child link="thruster_link_6"/>
-    <origin xyz="0 0 0.2" rpy="0 0 0"/>
-    <axis xyz="0 0 1"/>
-  </joint>
-  <link name="thruster_link_6"/>
-  <!-- ros2_control tag for hardware interface -->
-  <ros2_control name="scara_control" type="system">
-    <hardware>
-      <plugin>scara_simulator_layer/ScaraSimulatorInterface</plugin>
-    </hardware>
-    <joint name="thruster_joint_1">
-      <command_interface name="effort"/>
-      <state_interface name="effort"/>
-    </joint>
-    <joint name="thruster_joint_2">
-      <command_interface name="effort"/>
-      <state_interface name="effort"/>
-    </joint>
-    <joint name="thruster_joint_3">
-      <command_interface name="effort"/>
-      <state_interface name="effort"/>
-    </joint>
-    <joint name="thruster_joint_4">
-      <command_interface name="effort"/>
-      <state_interface name="effort"/>
-    </joint>
-  </ros2_control>
-</robot>
+/home/eia/repo/rbi_2025_2/scara/scara_ws/src/scara_mujoco_description/urdf/scara_description.urdf.xacro
