Commit message: genral docs: Fized spelling issues and added multiple images
dockerfiles: added some QOL imports

launch files: added some parameters for the user to get out of the box operation

File: abb/abb_ws/src/abb_gz_description/urdf/irb140_description.xacro (robot description, xacro)
@@ -1,181 +1,301 @@
-<?xml version="1.0" ?>
-<robot name="abb_irb140"
-       xmlns:xacro="http://ros.org/wiki/xacro">
-    <xacro:include filename="common_properties.xacro" />
-  <link name="base_link">
-    <visual>
-      <origin rpy="0 0 0" xyz="0 0 0"/>
-      <geometry>
-        <mesh filename="package://abb_gz_description/meshes/irb140/visual/base_link.stl"/>
-      </geometry>
-      <material name="abb_orange">
-        <color rgba="1 0.43 0 1"/>
-      </material>
-    </visual>
-    <collision>
-      <geometry>
-        <mesh filename="package://abb_gz_description/meshes/irb140/collision/base_link.stl"/>
-      </geometry>
-      <material name="yellow">
-        <color rgba="0 1 1 1"/>
-      </material>
-    </collision>
-    <xacro:box_inertia m="1000" x="0.5" y="0.5" z="0.5" o_xyz="0 0 0.2" o_rpy="0 0 0" />
-  </link>
-  <link name="link_1">
-    <visual>
-      <origin rpy="0 0 0" xyz="0 0 0"/>
-      <geometry>
-        <mesh filename="package://abb_gz_description/meshes/irb140/visual/link_1.stl"/>
-      </geometry>
-      <material name="abb_orange"/>
-    </visual>
-    <collision>
-      <origin rpy="0 0 0" xyz="0 0 0"/>
-      <geometry>
-        <mesh filename="package://abb_gz_description/meshes/irb140/collision/link_1.stl"/>
-      </geometry>
-      <material name="yellow"/>
-    </collision>
-    <xacro:cylinder_inertia m="1" r="0.15" l="0.5" o_xyz="0 0 0.25" o_rpy="0 0 0" />
-  </link>
-  <link name="link_2">
-    <visual>
-      <origin rpy="0 0 0" xyz="-0.28 0 -1.38"/>
-      <geometry>
-        <mesh filename="package://abb_gz_description/meshes/irb140/visual/link_2.stl"/>
-      </geometry>
-      <material name="abb_orange"/>
-    </visual>
-    <collision>
-      <origin rpy="0 0 0" xyz="-0.28 0 -1.38"/>
-      <geometry>
-        <mesh filename="package://abb_gz_description/meshes/irb140/collision/link_2.stl"/>
-      </geometry>
-      <material name="yellow"/>
-    </collision>
-    <xacro:box_inertia m="1" x="1.42" y="0.2" z="0.2" o_xyz="0.71 0 0" o_rpy="0 0 0" />
-  </link>
-  <link name="link_3">
-    <visual>
-      <origin rpy="0 0 0" xyz="-0.28 0 -2.8"/>
-      <geometry>
-        <mesh filename="package://abb_gz_description/meshes/irb140/visual/link_3.stl"/>
-      </geometry>
-      <material name="abb_orange"/>
-    </visual>
-    <collision>
-      <origin rpy="0 0 0" xyz="-0.28 0 -2.8"/>
-      <geometry>
-        <mesh filename="package://abb_gz_description/meshes/irb140/collision/link_3.stl"/>
-      </geometry>
-      <material name="yellow"/>
-    </collision>
-    <xacro:box_inertia m="1" x="1.49" y="0.15" z="0.15" o_xyz="0.745 0 0" o_rpy="0 0 0" />
-  </link>
-  <link name="link_4">
-    <visual>
-      <origin rpy="0 0 0" xyz="-0.28 0 -2.8"/>
-      <geometry>
-        <mesh filename="package://abb_gz_description/meshes/irb140/visual/link_4.stl"/>
-      </geometry>
-      <material name="abb_orange"/>
-    </visual>
-    <collision>
-      <origin rpy="0 0 0" xyz="-0.28 0 -2.8"/>
-      <geometry>
-        <mesh filename="package://abb_gz_description/meshes/irb140/collision/link_4.stl"/>
-      </geometry>
-      <material name="yellow"/>
-    </collision>
-    <xacro:box_inertia m="1" x="0.1" y="0.1" z="0.1" o_xyz="0 0 0" o_rpy="0 0 0" />
-  </link>
-  <link name="link_5">
-    <visual>
-      <origin rpy="0 0 0" xyz="-1.77 0 -2.8"/>
-      <geometry>
-        <mesh filename="package://abb_gz_description/meshes/irb140/visual/link_5.stl"/>
-      </geometry>
-      <material name="abb_orange"/>
-    </visual>
-    <collision>
-      <origin rpy="0 0 0" xyz="-1.77 0 -2.8"/>
-      <geometry>
-        <mesh filename="package://abb_gz_description/meshes/irb140/collision/link_5.stl"/>
-      </geometry>
-      <material name="yellow"/>
-    </collision>
-    <xacro:cylinder_inertia m="1" r="0.05" l="0.1" o_xyz="0 0 0" o_rpy="0 0 0" />
-  </link>
-  <link name="link_6">
-    <visual>
-      <origin rpy="0 0 0" xyz="-1.77 0 -2.8"/>
-      <geometry>
-        <mesh filename="package://abb_gz_description/meshes/irb140/visual/link_6.stl"/>
-      </geometry>
-      <material name="abb_orange"/>
-    </visual>
-    <collision>
-      <origin rpy="0 0 0" xyz="-1.77 0 -2.8"/>
-      <geometry>
-        <mesh filename="package://abb_gz_description/meshes/irb140/collision/link_6.stl"/>
-      </geometry>
-      <material name="yellow"/>
-    </collision>
-    <xacro:cylinder_inertia m="1" r="0.03" l="0.05" o_xyz="0 0 0" o_rpy="0 0 0" />
-  </link>
-  <link name="tool"/>
+<?xml version="1.0"?>
+<robot xmlns:xacro="http://www.ros.org/wiki/xacro" name="abb_robot">
+  <!-- Materials for visualization -->
+  <material name="red">
+    <color rgba="1 0 0 1"/>
+  </material>
+  <material name="blue">
+    <color rgba="0 0 1 1"/>
+  </material>
+  <!-- Base link (world reference) -->
+  <link name="world_0"/>
+  <!-- ABB Base Link -->
+  <link name="abb_base">
+    <visual>
+      <origin xyz="0 0 0" rpy="0 0 0"/>
+      <geometry>
+        <box size="0.6 0.6 0.1"/>
+      </geometry>
+      <material name="red"/>
+    </visual>
+    <collision>
+      <origin xyz="0 0 0" rpy="0 0 0"/>
+      <geometry>
+        <box size="0.6 0.6 0.1"/>
+      </geometry>
+    </collision>
+    <inertial>
+      <origin xyz="0 0 0" rpy="0 0 0"/>
+      <mass value="1000"/>
+      <inertia ixx="5.05" ixy="0.0" ixz="0.0" iyy="5.05" iyz="0.0" izz="10.0"/>
+    </inertial>
+  </link>
+  <joint name="world_to_base" type="fixed">
+    <parent link="world_0"/>
+    <child link="abb_base"/>
+    <origin xyz="0 0 0.05" rpy="0 0 0"/>
+  </joint>
+  <!-- First Joint Body -->
+  <link name="first_joint_body">
+    <visual>
+      <origin xyz="0 0 -0.245" rpy="0 0 0"/>
+      <geometry>
+        <cylinder radius="0.3" length="0.08"/>
+      </geometry>
+      <material name="blue"/>
+    </visual>
+    <visual>
+      <origin xyz="-0.245 0 0" rpy="0 0 0"/>
+      <geometry>
+        <box size="0.2 0.6 0.2"/>
+      </geometry>
+      <material name="red"/>
+    </visual>
+    <visual>
+      <origin xyz="0 0.25 0" rpy="0 0 0"/>
+      <geometry>
+        <box size="0.4 0.1 0.2"/>
+      </geometry>
+      <material name="red"/>
+    </visual>
+    <collision>
+      <origin xyz="0 0 -0.245" rpy="0 0 0"/>
+      <geometry>
+        <cylinder radius="0.3" length="0.08"/>
+      </geometry>
+    </collision>
+    <collision>
+      <origin xyz="-0.245 0 0" rpy="0 0 0"/>
+      <geometry>
+        <box size="0.2 0.6 0.2"/>
+      </geometry>
+    </collision>
+    <collision>
+      <origin xyz="0 0.25 0" rpy="0 0 0"/>
+      <geometry>
+        <box size="0.4 0.1 0.2"/>
+      </geometry>
+    </collision>
+    <inertial>
+      <origin xyz="0 0 0" rpy="0 0 0"/>
+      <mass value="10"/>
+      <inertia ixx="0.5" ixy="0.0" ixz="0.0" iyy="0.5" iyz="0.0" izz="0.8"/>
+    </inertial>
+  </link>
   <joint name="position_joint_0" type="revolute">
-    <origin rpy="0 0 0" xyz="0 0 0"/>
-    <parent link="base_link"/>
-    <child link="link_1"/>
-    <axis xyz="0 0 1"/>
-    <limit effort="100" lower="-3.1416" upper="3.1416" velocity="2.618"/>
-  </joint>
+    <parent link="abb_base"/>
+    <child link="first_joint_body"/>
+    <origin xyz="0 0 0.342" rpy="0 0 0"/>
+    <axis xyz="0 0 1"/>
+    <limit lower="-3.14159" upper="3.14159" effort="1000" velocity="2.0"/>
+    <dynamics damping="0.7" friction="0.0"/>
+  </joint>
+  <!-- Second Joint Body -->
+  <link name="second_joint_body">
+    <visual>
+      <origin xyz="0 0 0" rpy="0 0 0"/>
+      <geometry>
+        <cylinder radius="0.1" length="0.4"/>
+      </geometry>
+      <material name="blue"/>
+    </visual>
+    <visual>
+      <origin xyz="0.2 0 0.25" rpy="0 0 0"/>
+      <geometry>
+        <box size="0.6 0.2 0.1"/>
+      </geometry>
+      <material name="red"/>
+    </visual>
+    <collision>
+      <origin xyz="0 0 0" rpy="0 0 0"/>
+      <geometry>
+        <cylinder radius="0.1" length="0.4"/>
+      </geometry>
+    </collision>
+    <collision>
+      <origin xyz="0.2 0 0.25" rpy="0 0 0"/>
+      <geometry>
+        <box size="0.6 0.2 0.1"/>
+      </geometry>
+    </collision>
+    <inertial>
+      <origin xyz="0.2 0 0.25" rpy="0 0 0"/>
+      <mass value="8"/>
+      <inertia ixx="0.3" ixy="0.0" ixz="0.0" iyy="0.5" iyz="0.0" izz="0.4"/>
+    </inertial>
+  </link>
   <joint name="position_joint_1" type="revolute">
-    <origin rpy="0 0 0" xyz="0.28 0 1.38"/>
-    <parent link="link_1"/>
-    <child link="link_2"/>
-    <axis xyz="0 1 0"/>
-    <limit effort="100" lower="-1.7453" upper="1.9199" velocity="2.618"/>
-  </joint>
+    <parent link="first_joint_body"/>
+    <child link="second_joint_body"/>
+    <origin xyz="0.06988 0 0" rpy="1.5708 -1.5708 0"/>
+    <axis xyz="0 0 1"/>
+    <limit lower="-3.14159" upper="3.14159" effort="1000" velocity="2.0"/>
+    <dynamics damping="0.7" friction="0.0"/>
+  </joint>
+  <!-- Third Joint Body -->
+  <link name="third_joint_body">
+    <visual>
+      <origin xyz="0 0 0" rpy="0 0 0"/>
+      <geometry>
+        <cylinder radius="0.1" length="0.4"/>
+      </geometry>
+      <material name="blue"/>
+    </visual>
+    <collision>
+      <origin xyz="0 0 0" rpy="0 0 0"/>
+      <geometry>
+        <cylinder radius="0.1" length="0.4"/>
+      </geometry>
+    </collision>
+    <inertial>
+      <origin xyz="0 0 0" rpy="0 0 0"/>
+      <mass value="5"/>
+      <inertia ixx="0.15" ixy="0.0" ixz="0.0" iyy="0.15" iyz="0.0" izz="0.05"/>
+    </inertial>
+  </link>
   <joint name="position_joint_2" type="revolute">
-    <origin rpy="0 0 0" xyz="0 0 1.42"/>
-    <parent link="link_2"/>
-    <child link="link_3"/>
-    <axis xyz="0 1 0"/>
-    <limit effort="100" lower="-1.0472" upper="1.1345" velocity="2.618"/>
-  </joint>
+    <parent link="second_joint_body"/>
+    <child link="third_joint_body"/>
+    <origin xyz="0.362 0 0" rpy="0 0 3.14159"/>
+    <axis xyz="0 0 1"/>
+    <limit lower="-3.14159" upper="3.14159" effort="1000" velocity="2.0"/>
+    <dynamics damping="0.7" friction="0.0"/>
+  </joint>
+  <!-- Fourth Joint Body -->
+  <link name="fourth_joint_body">
+    <visual>
+      <origin xyz="0 0 0.155" rpy="0 0 0"/>
+      <geometry>
+        <cylinder radius="0.08" length="0.2"/>
+      </geometry>
+      <material name="blue"/>
+    </visual>
+    <collision>
+      <origin xyz="0 0 0.155" rpy="0 0 0"/>
+      <geometry>
+        <cylinder radius="0.08" length="0.2"/>
+      </geometry>
+    </collision>
+    <inertial>
+      <origin xyz="0 0 0.155" rpy="0 0 0"/>
+      <mass value="3"/>
+      <inertia ixx="0.05" ixy="0.0" ixz="0.0" iyy="0.05" iyz="0.0" izz="0.02"/>
+    </inertial>
+  </link>
   <joint name="position_joint_3" type="revolute">
-    <origin rpy="0 0 0" xyz="0 0 0"/>
-    <parent link="link_3"/>
-    <child link="link_4"/>
-    <axis xyz="1 0 0"/>
-    <limit effort="100" lower="-3.49" upper="3.49" velocity="6.2832"/>
-  </joint>
+    <parent link="third_joint_body"/>
+    <child link="fourth_joint_body"/>
+    <origin xyz="0 0.380 0" rpy="-1.5708 0 3.14159"/>
+    <axis xyz="0 0 1"/>
+    <limit lower="-3.14159" upper="3.14159" effort="1000" velocity="2.0"/>
+    <dynamics damping="0.5" friction="0.0"/>
+  </joint>
+  <!-- Fifth Joint Body -->
+  <link name="fifth_joint_body">
+    <visual>
+      <origin xyz="0 0 0" rpy="0 0 0"/>
+      <geometry>
+        <cylinder radius="0.05" length="0.2"/>
+      </geometry>
+      <material name="blue"/>
+    </visual>
+    <collision>
+      <origin xyz="0 0 0" rpy="0 0 0"/>
+      <geometry>
+        <cylinder radius="0.05" length="0.2"/>
+      </geometry>
+    </collision>
+    <inertial>
+      <origin xyz="0 0 0" rpy="0 0 0"/>
+      <mass value="2"/>
+      <inertia ixx="0.02" ixy="0.0" ixz="0.0" iyy="0.02" iyz="0.0" izz="0.01"/>
+    </inertial>
+  </link>
   <joint name="position_joint_4" type="revolute">
-    <origin rpy="0 0 0" xyz="1.49 0 0"/>
-    <parent link="link_4"/>
-    <child link="link_5"/>
-    <axis xyz="0 1 0"/>
-    <limit effort="100" lower="-2.0944" upper="2.0944" velocity="6.2832"/>
-  </joint>
+    <parent link="fourth_joint_body"/>
+    <child link="fifth_joint_body"/>
+    <origin xyz="0 0 0" rpy="-1.5708 0 3.14159"/>
+    <axis xyz="0 0 1"/>
+    <limit lower="-3.14159" upper="3.14159" effort="1000" velocity="2.0"/>
+    <dynamics damping="0.5" friction="0.0"/>
+  </joint>
+  <!-- Sixth Joint Body (End Effector) -->
+  <link name="sixth_joint_body">
+    <visual>
+      <origin xyz="0 0 0.05" rpy="0 0 0"/>
+      <geometry>
+        <cylinder radius="0.02" length="0.1"/>
+      </geometry>
+      <material name="blue"/>
+    </visual>
+    <collision>
+      <origin xyz="0 0 0.05" rpy="0 0 0"/>
+      <geometry>
+        <cylinder radius="0.02" length="0.1"/>
+      </geometry>
+    </collision>
+    <inertial>
+      <origin xyz="0 0 0.05" rpy="0 0 0"/>
+      <mass value="0.5"/>
+      <inertia ixx="0.001" ixy="0.0" ixz="0.0" iyy="0.001" iyz="0.0" izz="0.0005"/>
+    </inertial>
+  </link>
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
File: abb/abb_ws/src/abb_mujoco_description/urdf/abb_description.urdf.xacro (robot description, xacro)
@@ -1,69 +1,161 @@
 <?xml version="1.0"?>
-<robot name="rover" xmlns:xacro="http://www.ros.org/wiki/xacro">
-  <!-- Main body -->
-  <link name="hull_link">
+<robot xmlns:xacro="http://www.ros.org/wiki/xacro" name="abb_robot">
+  <!-- Materials for visualization -->
+  <material name="red">
+    <color rgba="1 0 0 1"/>
+  </material>
+  <material name="blue">
+    <color rgba="0 0 1 1"/>
+  </material>
+  <material name="grey">
+    <color rgba="0.5 0.5 0.5 1"/>
+  </material>
+  <!-- Base link (world reference) -->
+  <link name="world_0"/>
+  <!-- ABB Base Link -->
+  <link name="abb_base">
     <visual>
+      <origin xyz="0 0 0" rpy="0 0 0"/>
       <geometry>
-        <box size="0.6 0.4 0.2"/>
+        <box size="0.6 0.6 0.1"/>
       </geometry>
-      <material name="blue">
-        <color rgba="0.1 0.1 0.8 1"/>
-      </material>
+      <material name="red"/>
     </visual>
-    <collision>
+  </link>
+  <joint name="world_to_base" type="fixed">
+    <parent link="world_0"/>
+    <child link="abb_base"/>
+    <origin xyz="0 0 0.05" rpy="0 0 0"/>
+  </joint>
+  <!-- First Joint Body -->
+  <link name="first_joint_body">
+    <visual>
+      <origin xyz="0 0 -0.245" rpy="0 0 0"/>
       <geometry>
-        <box size="0.6 0.4 0.2"/>
+        <cylinder radius="0.3" length="0.08"/>
       </geometry>
-    </collision>
-    <inertial>
-      <mass value="10"/>
-      <origin xyz="0 0 0"/>
-      <inertia ixx="1" ixy="0" ixz="0" iyy="1" iyz="0" izz="1"/>
-    </inertial>
+      <material name="blue"/>
+    </visual>
+    <visual>
+      <origin xyz="-0.245 0 0" rpy="0 0 0"/>
+      <geometry>
+        <box size="0.2 0.6 0.2"/>
+      </geometry>
+      <material name="red"/>
+    </visual>
+    <visual>
+      <origin xyz="0 0.25 0" rpy="0 0 0"/>
+      <geometry>
+        <box size="0.4 0.1 0.2"/>
+      </geometry>
+      <material name="red"/>
+    </visual>
   </link>
-  <!-- Six thruster joints (effort controlled) -->
-  <!-- X, Y, Z, Roll, Pitch, Yaw -->
-  <joint name="thruster_joint_1" type="continuous">
-    <parent link="hull_link"/>
-    <child link="thruster_link_1"/>
-    <origin xyz="0.3 0 0" rpy="0 0 0"/>
-    <axis xyz="1 0 0"/>
+  <joint name="position_joint_0" type="revolute">
+    <parent link="abb_base"/>
+    <child link="first_joint_body"/>
+    <origin xyz="0 0 0.342" rpy="0 0 0"/>
+    <axis xyz="0 0 1"/>
+     <limit lower="-3.14159" upper="3.14159" effort="1000" velocity="2.0"/>
   </joint>
-  <link name="thruster_link_1"/>
-  <joint name="thruster_joint_2" type="continuous">
-    <parent link="hull_link"/>
-    <child link="thruster_link_2"/>
-    <origin xyz="-0.3 0 0" rpy="0 0 0"/>
-    <axis xyz="0 1 0"/>
+  <!-- Second Joint Body -->
+  <link name="second_joint_body">
+    <visual>
+      <origin xyz="0 0 0" rpy="0 0 0"/>
+      <geometry>
+        <cylinder radius="0.1" length="0.4"/>
+      </geometry>
+      <material name="blue"/>
+    </visual>
+    <visual>
+      <origin xyz="0.2 0 0.25" rpy="0 0 0"/>
+      <geometry>
+        <box size="0.6 0.2 0.1"/>
+      </geometry>
+      <material name="red"/>
+    </visual>
+  </link>
+  <joint name="position_joint_1" type="revolute">
+    <parent link="first_joint_body"/>
+    <child link="second_joint_body"/>
+    <origin xyz="0.06988 0 0" rpy="1.5708 -1.5708 0"/>
+    <axis xyz="0 0 1"/>
+     <limit lower="-3.14159" upper="3.14159" effort="1000" velocity="2.0"/>
   </joint>
-  <link name="thruster_link_2"/>
-  <joint name="thruster_joint_3" type="continuous">
-    <parent link="hull_link"/>
-    <child link="thruster_link_3"/>
-    <origin xyz="0 0 0.1" rpy="0 0 0"/>
+  <!-- Third Joint Body -->
+  <link name="third_joint_body">
+    <visual>
+      <origin xyz="0 0 0" rpy="0 0 0"/>
+      <geometry>
+        <cylinder radius="0.1" length="0.4"/>
+      </geometry>
+      <material name="blue"/>
+    </visual>
+  </link>
+  <joint name="position_joint_2" type="revolute">
+    <parent link="second_joint_body"/>
+    <child link="third_joint_body"/>
+    <origin xyz="0.362 0 0" rpy="0 0 3.14159"/>
     <axis xyz="0 0 1"/>
+     <limit lower="-3.14159" upper="3.14159" effort="1000" velocity="2.0"/>
   </joint>
-  <link name="thruster_link_3"/>
-  <joint name="thruster_joint_4" type="continuous">
-    <parent link="hull_link"/>
-    <child link="thruster_link_4"/>
-    <origin xyz="0 0.2 0" rpy="0 0 0"/>
-    <axis xyz="1 0 0"/>
+  <!-- Fourth Joint Body -->
+  <link name="fourth_joint_body">
+    <visual>
+      <origin xyz="0 0 0.155" rpy="0 0 0"/>
+      <geometry>
+        <cylinder radius="0.08" length="0.2"/>
+      </geometry>
+      <material name="blue"/>
+    </visual>
+  </link>
+  <joint name="position_joint_3" type="revolute">
+    <parent link="third_joint_body"/>
+    <child link="fourth_joint_body"/>
+    <origin xyz="0 0.380 0" rpy="-1.5708 0 3.14159"/>
+    <axis xyz="0 0 1"/>
+     <limit lower="-3.14159" upper="3.14159" effort="1000" velocity="2.0"/>
   </joint>
-  <link name="thruster_link_4"/>
-  <joint name="thruster_joint_5" type="continuous">
-    <parent link="hull_link"/>
-    <child link="thruster_link_5"/>
-    <origin xyz="0 -0.2 0" rpy="0 0 0"/>
-    <axis xyz="0 1 0"/>
+  <!-- Fifth Joint Body -->
+  <link name="fifth_joint_body">
+    <visual>
+      <origin xyz="0 0 0" rpy="0 0 0"/>
+      <geometry>
+        <cylinder radius="0.05" length="0.2"/>
+      </geometry>
+      <material name="blue"/>
+    </visual>
+  </link>
+  <joint name="position_joint_4" type="revolute">
+    <parent link="fourth_joint_body"/>
+    <child link="fifth_joint_body"/>
+    <origin xyz="0 0 0" rpy="-1.5708 0 3.14159"/>
+    <axis xyz="0 0 1"/>
+     <limit lower="-3.14159" upper="3.14159" effort="1000" velocity="2.0"/>
   </joint>
-  <link name="thruster_link_5"/>
-  <joint name="thruster_joint_6" type="continuous">
-    <parent link="hull_link"/>
-    <child link="thruster_link_6"/>
-    <origin xyz="0 0 0.2" rpy="0 0 0"/>
+  <!-- Sixth Joint Body (End Effector) -->
+  <link name="sixth_joint_body">
+    <visual>
+      <origin xyz="0 0 0.05" rpy="0 0 0"/>
+      <geometry>
+        <cylinder radius="0.02" length="0.1"/>
+      </geometry>
+      <material name="blue"/>
+    </visual>
+  </link>
+  <joint name="position_joint_5" type="revolute">
+    <parent link="fifth_joint_body"/>
+    <child link="sixth_joint_body"/>
+    <origin xyz="0 0.25 0" rpy="-1.5708 0 3.14159"/>
     <axis xyz="0 0 1"/>
+     <limit lower="-3.14159" upper="3.14159" effort="1000" velocity="2.0"/>
   </joint>
-  <link name="thruster_link_6"/>
+  <!-- End Effector Link (for TCP) -->
+  <link name="tool"/>
+  <joint name="tool_joint" type="fixed">
+    <parent link="sixth_joint_body"/>
+    <child link="tool"/>
+    <origin xyz="0 0 0" rpy="0 0 0"/>
+  </joint>
   <!-- ros2_control tag for hardware interface -->
   <ros2_control name="abb_control" type="system">

File: scara/scara_ws/src/scara_mujoco_description/urdf/scara_description.xacro (robot description, xacro)
@@ -8,9 +8,4 @@
   <!-- ============== Base ============== -->
   <link name="world_0">
-    <inertial>
-      <origin xyz="0 0 0" rpy="0 0 0"/>
-      <mass value="10000.0"/>
-      <inertia ixx="0.002" ixy="0" ixz="0" iyy="0.002" iyz="0" izz="0.002"/>
-    </inertial>
     <visual>
       <origin xyz="0 0 0" rpy="0 0 0"/>
